Commit message: Renamed node and added visualization node

File: src/pendulum_sim/urdf/pendulum.urdf (robot description, URDF)
Before this commit: robot single_link_arm, 3 links, 2 joints
Links:
- link base: geometry collision cylinder length=0.42 radius=.075; visual mesh filename=package://pendulum_sim/models/Base_2.stl
- link link1: geometry collision cylinder length=0.36 radius=.05; visual mesh filename=package://pendulum_sim/models/Arm_2.stl
